Commit message: Zoe2 xacro now successfully launches.

File: cmu_zoe2/zoe2_description/urdf/common/axle.xacro (robot description, xacro)
@@ -1,5 +1,5 @@
 <?xml version="1.0"?>
 <robot xmlns:xacro="http://www.ros.org/wiki/xacro" name="robot">
-    <xacro:macro name="hinge" params="name rpy xyz" >
+    <xacro:macro name="axle" params="name rpy xyz" >
         <link
             name="${name}">
@@ -9,12 +9,12 @@
                     rpy="${rpy}" />
                 <mass
-                    value="1.60265212368031" />
+                    value="2.76276470983555" />
                 <inertia
-                    ixx="0.00789007052519473"
-                    ixy="-4.51083375595945E-06"
-                    ixz="-3.52376942846933E-05"
-                    iyy="0.00778556714593041"
-                    iyz="1.5780343532552E-06"
-                    izz="0.00273377335912292" />
+                    ixx="0.0151578893043941"
+                    ixy="-6.10514243326588E-15"
+                    ixz="-8.69280987887411E-16"
+                    iyy="0.615173226679267"
+                    iyz="-9.50117240753409E-16"
+                    izz="0.620920397735107" />
             </inertial>
             <visual>
@@ -24,10 +24,10 @@
                 <geometry>
                     <mesh
-                        filename="file://$(find zoe2_description)/description/meshes/zoe2/collision/back_hinge.STL" />
+                        filename="file://$(find zoe2_description)/meshes/zoe2/collision/front_axle.STL" />
                 </geometry>
                 <material
                     name="">
                     <color
-                        rgba="0.866666666666667 0.909803921568627 1 1" />
+                        rgba="0.529411764705882 0.549019607843137 0.549019607843137 1" />
                 </material>
             </visual>
@@ -38,5 +38,5 @@
                 <geometry>
                     <mesh
-                        filename="file://$(find zoe2_description)/description/meshes/zoe2/collision/back_hinge.STL" />
+                        filename="file://$(find zoe2_description)/meshes/zoe2/collision/front_axle.STL" />
                 </geometry>
             </collision>

File: cmu_zoe2/zoe2_description/urdf/common/chassis.xacro (robot description, xacro)
@@ -1,5 +1,5 @@
 <?xml version="1.0"?>
 <robot xmlns:xacro="http://www.ros.org/wiki/xacro" name="robot">
-    <xacro:macro name="wheel" params="name rpy xyz">
+    <xacro:macro name="chassis" params="name rpy xyz">
         <link
             name="${name}">
@@ -9,12 +9,12 @@
                     rpy="${rpy}" />
                 <mass
-                    value="32.3144669983568" />
+                    value="651.498299444812" />
                 <inertia
-                    ixx="1.03582581735133"
-                    ixy="3.69335039891439E-06"
-                    ixz="9.72371372309766E-09"
-                    iyy="1.97706054850814"
-                    iyz="-4.49800950049796E-08"
-                    izz="1.03582581231329" />
+                    ixx="149.816150034198"
+                    ixy="2.25656686320975E-10"
+                    ixz="1.4248945896711E-08"
+                    iyy="204.954522277079"
+                    iyz="-0.376718299070616"
+                    izz="79.5488628930089" />
             </inertial>
             <visual>
@@ -24,10 +24,10 @@
                 <geometry>
                     <mesh
-                        filename="file://$(find zoe2_description)/description/meshes/zoe2/collision/back_right_wheel.STL" />
+                        filename="file://$(find zoe2_description)/meshes/zoe2/collision/chassis.STL" />
                 </geometry>
                 <material
                     name="">
                     <color
-                        rgba="0.294117647058824 0.294117647058824 0.294117647058824 1" />
+                        rgba="0.866666666666667 0.909803921568627 1 1" />
                 </material>
             </visual>
@@ -38,5 +38,5 @@
                 <geometry>
                     <mesh
-                        filename="file://$(find zoe2_description)/description/meshes/zoe2/collision/back_right_wheel.STL" />
+                        filename="file://$(find zoe2_description)/meshes/zoe2/collision/chassis.STL" />
                 </geometry>
             </collision>

File: cmu_zoe2/zoe2_description/urdf/common/hinge.xacro (robot description, xacro)
@@ -1,5 +1,5 @@
 <?xml version="1.0"?>
 <robot xmlns:xacro="http://www.ros.org/wiki/xacro" name="robot">
-    <xacro:macro name="chassis" params="name rpy xyz">
+    <xacro:macro name="hinge" params="name rpy xyz" >
         <link
             name="${name}">
@@ -9,12 +9,12 @@
                     rpy="${rpy}" />
                 <mass
-                    value="651.498299444812" />
+                    value="1.60265212368031" />
                 <inertia
-                    ixx="149.816150034198"
-                    ixy="2.25656686320975E-10"
-                    ixz="1.4248945896711E-08"
-                    iyy="204.954522277079"
-                    iyz="-0.376718299070616"
-                    izz="79.5488628930089" />
+                    ixx="0.00789007052519473"
+                    ixy="-4.51083375595945E-06"
+                    ixz="-3.52376942846933E-05"
+                    iyy="0.00778556714593041"
+                    iyz="1.5780343532552E-06"
+                    izz="0.00273377335912292" />
             </inertial>
             <visual>
@@ -24,5 +24,5 @@
                 <geometry>
                     <mesh
-                        filename="file://$(find zoe2_description)/description/meshes/zoe2/collision/chassis.STL" />
+                        filename="file://$(find zoe2_description)/meshes/zoe2/collision/back_hinge.STL" />
                 </geometry>
                 <material
@@ -38,5 +38,5 @@
                 <geometry>
                     <mesh
-                        filename="file://$(find zoe2_description)/description/meshes/zoe2/collision/chassis.STL" />
+                        filename="file://$(find zoe2_description)/meshes/zoe2/collision/back_hinge.STL" />
                 </geometry>
             </collision>

File: cmu_zoe2/zoe2_description/urdf/common/wheel.xacro (robot description, xacro)
@@ -1,5 +1,5 @@
 <?xml version="1.0"?>
 <robot xmlns:xacro="http://www.ros.org/wiki/xacro" name="robot">
-    <xacro:macro name="axle" params="name rpy xyz" >
+    <xacro:macro name="wheel" params="name rpy xyz">
         <link
             name="${name}">
@@ -9,12 +9,12 @@
                     rpy="${rpy}" />
                 <mass
-                    value="2.76276470983555" />
+                    value="32.3144669983568" />
                 <inertia
-                    ixx="0.0151578893043941"
-                    ixy="-6.10514243326588E-15"
-                    ixz="-8.69280987887411E-16"
-                    iyy="0.615173226679267"
-                    iyz="-9.50117240753409E-16"
-                    izz="0.620920397735107" />
+                    ixx="1.03582581735133"
+                    ixy="3.69335039891439E-06"
+                    ixz="9.72371372309766E-09"
+                    iyy="1.97706054850814"
+                    iyz="-4.49800950049796E-08"
+                    izz="1.03582581231329" />
             </inertial>
             <visual>
@@ -24,10 +24,10 @@
                 <geometry>
                     <mesh
-                        filename="file://$(find zoe2_description)/description/meshes/zoe2/collision/front_axle.STL" />
+                        filename="file://$(find zoe2_description)/meshes/zoe2/collision/back_right_wheel.STL" />
                 </geometry>
                 <material
                     name="">
                     <color
-                        rgba="0.529411764705882 0.549019607843137 0.549019607843137 1" />
+                        rgba="0.294117647058824 0.294117647058824 0.294117647058824 1" />
                 </material>
             </visual>
@@ -38,5 +38,5 @@
                 <geometry>
                     <mesh
-                        filename="file://$(find zoe2_description)/description/meshes/zoe2/collision/front_axle.STL" />
+                        filename="file://$(find zoe2_description)/meshes/zoe2/collision/back_right_wheel.STL" />
                 </geometry>
             </collision>

File: cmu_zoe2/zoe2_description/urdf/zoe2/zoe2_macro.ros2_control.xacro (robot description, xacro)
@@ -36,24 +36,20 @@
           <state_interface name="position" />
           <state_interface name="velocity" />
-          <command_interface
-              name="velocity" />
+          <command_interface name="velocity" />
       </joint>
       <joint name="front_right_hinge_joint">
           <state_interface name="position" />
           <state_interface name="velocity" />
-          <command_interface
-              name="velocity" />
+          <command_interface name="velocity" />
       </joint>
       <joint name="back_right_hinge_joint">
           <state_interface name="position" />
           <state_interface name="velocity" />
-          <command_interface
-              name="velocity" />
+          <command_interface name="velocity" />
       </joint>
       <joint name="back_left_hinge_joint">
           <state_interface name="position" />
           <state_interface name="velocity" />
-          <command_interface
-              name="velocity" />
+          <command_interface name="velocity" />
       </joint>
     </ros2_control>

File: cmu_zoe2/zoe2_description/urdf/zoe2/zoe2_macro.xacro (robot description, xacro)
@@ -3,17 +3,11 @@
   <xacro:include filename="$(find zoe2_description)/urdf/common/inertials.xacro" />
   <xacro:include filename="$(find zoe2_description)/urdf/common/materials.xacro" />
-  <xacro:include filename="$(find zoe2_description)/urdf/components/wheel.xacro" />
-  <xacro:include filename="$(find zoe2_description)/urdf/components/chassis.xacro" />
-  <xacro:include filename="$(find zoe2_description)/urdf/components/axle.xacro" />
-  <xacro:include filename="$(find zoe2_description)/urdf/components/hinge.xacro" />
-  <xacro:include filename="$(find zoe2_description)/urdf/components/params.xacro" />
+  <xacro:include filename="$(find zoe2_description)/urdf/common/wheel.xacro" />
+  <xacro:include filename="$(find zoe2_description)/urdf/common/chassis.xacro" />
+  <xacro:include filename="$(find zoe2_description)/urdf/common/axle.xacro" />
+  <xacro:include filename="$(find zoe2_description)/urdf/common/hinge.xacro" />
+  <xacro:include filename="$(find zoe2_description)/urdf/common/params.xacro" />
   <xacro:macro name="zoe2" params="prefix parent *origin">
-    <link name="base_link">
-    </link>
-    <joint name="base_joint" type="fixed">
-        <parent link="base_link" />
-        <child link="chassis" />
-        <origin xyz="0 0 ${wheel_radius}" />
-    </joint>
+    <!-- LINKS -->
     <xacro:chassis name="chassis" rpy="0 0 0" xyz="0 0 0" />
     <xacro:hinge name="front_roll" rpy="${pi/2} 0 0" xyz="0 0 0" />
@@ -21,4 +15,26 @@
     <xacro:wheel name="front_left_wheel" rpy="0 0 ${-pi/2}" xyz="0 0 0" />
     <xacro:axle name="front_axle" rpy="${pi/2} 0 0" xyz="0 0 0" />
+    <xacro:wheel name="back_right_wheel" rpy="0 0 ${pi/2}" xyz="0 0 0" />
+    <xacro:wheel name="back_left_wheel" rpy="0 0 ${-pi/2}" xyz="0 0 0" />
+    <xacro:axle name="back_axle" rpy="${pi/2} 0 0" xyz="0 0 0" />
+    <xacro:hinge name="back_roll" rpy="${-pi/2} 0 0" xyz="0 0 0" />
+    <!-- END LINKS -->
+    <!-- JOINTS -->
+    <!-- base_joint fixes base_link to the environment -->
+    <!-- <joint name="${prefix}base_joint" type="fixed">
+        <xacro:insert_block name="origin" />
+        <parent link="${parent}" />
+        <child link="base_link" />
+        </joint>
+    <joint name="body_joint" type="fixed">
+        <parent link="base_link" />
+        <child link="chassis" />
+        <origin xyz="0 0 ${wheel_radius}" />
+    </joint> -->
+    <joint name="${prefix}base_joint" type="fixed">
+        <xacro:insert_block name="origin" />
+        <parent link="${parent}" />
+        <child link="chassis" />
+    </joint>
     <joint name="chassis_front_roll_joint" type="fixed">
         <parent link="chassis" />
@@ -45,9 +61,4 @@
         <axis xyz="1 0 0" />
     </joint>
-    <!-- @@@@@@@@@@@@@@@@@@@@@@@@@@@@@@@@@@@@@@@ -->
-    <xacro:wheel name="back_right_wheel" rpy="0 0 ${pi/2}" xyz="0 0 0" />
-    <xacro:wheel name="back_left_wheel" rpy="0 0 ${-pi/2}" xyz="0 0 0" />
-    <xacro:axle name="back_axle" rpy="${pi/2} 0 0" xyz="0 0 0" />
-    <xacro:hinge name="back_roll" rpy="${-pi/2} 0 0" xyz="0 0 0" />
     <joint name="back_roll_back_axle_joint" type="revolute">
         <parent link="back_roll" />
@@ -74,4 +85,5 @@
         <origin xyz="0 ${+(robot_length/2 - robot_hinge_length)} 0" />
     </joint>
+    <!-- END JOINTS -->
   </xacro:macro>
 </robot>
