Commit message: Added simple primitives for URDF collisions

File: zoe2_description/urdf/common/axle.xacro (robot description, xacro)
@@ -37,6 +37,7 @@
                     rpy="${rpy}" />
                 <geometry>
-                    <mesh
-                        filename="file://$(find zoe2_description)/meshes/zoe2/collision/front_axle.STL" />
+                    <!-- <mesh
+                        filename="file://$(find zoe2_description)/meshes/zoe2/collision/front_axle.STL" /> -->
+                    <box size="${axle_length} ${axle_box_width} ${axle_box_width}" />
                 </geometry>
             </collision>

File: zoe2_description/urdf/common/chassis.xacro (robot description, xacro)
@@ -34,9 +34,10 @@
             <collision>
                 <origin
-                    xyz="${xyz}"
+                    xyz="0 0 ${chassis_height/2-axle_box_width/2}"
                     rpy="${rpy}" />
                 <geometry>
-                    <mesh
-                        filename="file://$(find zoe2_description)/meshes/zoe2/collision/chassis.STL" />
+                    <!-- <mesh
+                        filename="file://$(find zoe2_description)/meshes/zoe2/collision/chassis.STL" /> -->
+                    <box size="${chassis_width} ${chassis_length} ${chassis_height}" />
                 </geometry>
             </collision>

File: zoe2_description/urdf/common/hinge.xacro (robot description, xacro)
@@ -37,6 +37,7 @@
                     rpy="${rpy}" />
                 <geometry>
-                    <mesh
-                        filename="file://$(find zoe2_description)/meshes/zoe2/collision/back_hinge.STL" />
+                    <!-- <mesh
+                        filename="file://$(find zoe2_description)/meshes/zoe2/collision/back_hinge.STL" /> -->
+                    <box size="${axle_box_width} ${axle_box_width} ${robot_hinge_length*2}" />
                 </geometry>
             </collision>

File: zoe2_description/urdf/common/params.xacro (robot description, xacro)
@@ -4,6 +4,17 @@
     <xacro:property name="robot_width" value="1.875" />
     <xacro:property name="robot_length" value="2"/>
+    <xacro:property name="base_link_height" value="0.4"/>
+    <!-- Chassis -->
+    <xacro:property name="chassis_length" value="1.5"/>
+    <xacro:property name="chassis_width" value="1.2"/>
+    <xacro:property name="chassis_height" value="0.5"/>
+    <!-- Hinge -->
     <xacro:property name="robot_hinge_length" value="0.2"/>
     <xacro:property name="front_vertical_limit" value="${pi/4}"/>
-    <xacro:property name="wheel_radius" value="0.4"/>
+    <!-- Wheel -->
+    <xacro:property name="wheel_radius" value="0.325"/>
+    <xacro:property name="wheel_thickness" value="0.05"/>
+    <!-- Axle -->
+    <xacro:property name="axle_box_width" value="0.1"/>
+    <xacro:property name="axle_length" value="${robot_width-wheel_thickness}"/>
 </robot>

File: zoe2_description/urdf/common/wheel.xacro (robot description, xacro)
@@ -35,8 +35,9 @@
                 <origin
                     xyz="${xyz}"
-                    rpy="${rpy}" />
+                    rpy="0 ${-pi/2} 0" />
                 <geometry>
-                    <mesh
-                        filename="file://$(find zoe2_description)/meshes/zoe2/collision/back_right_wheel.STL" />
+                    <!-- <mesh
+                        filename="file://$(find zoe2_description)/meshes/zoe2/collision/back_right_wheel.STL" /> -->
+                  <cylinder radius="${wheel_radius}" length="${wheel_thickness}"/>
                 </geometry>
             </collision>

File: zoe2_description/urdf/zoe2/zoe2_macro.xacro (robot description, xacro)
@@ -28,5 +28,5 @@
         <parent link="${prefix}base_link" />
         <child link="${prefix}chassis" />
-        <origin xyz="0 0 ${wheel_radius}" />
+        <origin xyz="0 0 ${base_link_height}" />
     </joint>
     <joint name="${prefix}chassis_front_roll_joint" type="fixed">

Commit message: Corrected dimensions of URDF file and controller to match those reported in https://ieeexplore.ieee.org/stamp/stamp.jsp?arnumber=6094930

File: zoe2_description/urdf/common/axle.xacro (robot description, xacro)
@@ -20,5 +20,5 @@
             <visual>
                 <origin
-                    xyz="${xyz}"
+                    xyz="0 0 -0.075"
                     rpy="${rpy}" />
                 <geometry>

File: zoe2_description/urdf/common/params.xacro (robot description, xacro)
@@ -2,6 +2,6 @@
     <robot xmlns:xacro="http://www.ros.org/wiki/xacro"  name="robot">
     <!-- all are in meters -->
-    <xacro:property name="robot_width" value="1.875" />
-    <xacro:property name="robot_length" value="2"/>
+    <xacro:property name="robot_width" value="1.64" />
+    <xacro:property name="robot_length" value="1.91"/>
     <xacro:property name="base_link_height" value="0.4"/>
     <!-- Chassis -->
@@ -18,3 +18,4 @@
     <xacro:property name="axle_box_width" value="0.1"/>
     <xacro:property name="axle_length" value="${robot_width-wheel_thickness}"/>
+    <xacro:property name="axle_drop" value="0.119"/>
 </robot>

File: zoe2_description/urdf/zoe2/zoe2_macro.xacro (robot description, xacro)
@@ -60,5 +60,5 @@
         <parent link="${prefix}front_roll" />
         <child link="${prefix}front_axle" />
-        <origin xyz="0 ${-robot_hinge_length} -0.075" />
+        <origin xyz="0 ${-robot_hinge_length} 0" />
         <axis xyz="0 0 1"/>
         <limit lower="${-front_vertical_limit}" upper="${front_vertical_limit}" effort="10" velocity="10"/>
@@ -67,5 +67,5 @@
         <parent link="${prefix}front_axle" />
         <child link="${prefix}front_right_wheel" />
-        <origin xyz="${robot_width/2} 0 0" />
+        <origin xyz="${robot_width/2} 0 -${axle_drop}" />
         <axis xyz="1 0 0" />
     </joint>
@@ -73,5 +73,5 @@
         <parent link="${prefix}front_axle" />
         <child link="${prefix}front_left_wheel" />
-        <origin xyz="${-robot_width/2} 0 0" />
+        <origin xyz="${-robot_width/2} 0 -${axle_drop}" />
         <axis xyz="1 0 0" />
     </joint>
@@ -80,5 +80,5 @@
         <parent link="${prefix}back_roll" />
         <child link="${prefix}back_axle" />
-        <origin xyz="0 ${robot_hinge_length} -0.075" />
+        <origin xyz="0 ${robot_hinge_length} 0" />
         <limit lower="${-front_vertical_limit}" upper="${front_vertical_limit}" effort="10" velocity="10"/>
         <axis xyz="0 0 1"/>
@@ -87,5 +87,5 @@
         <parent link="${prefix}back_axle" />
         <child link="${prefix}back_right_wheel" />
-        <origin xyz="${robot_width/2} 0 0" />
+        <origin xyz="${robot_width/2} 0 -${axle_drop}" />
         <axis xyz="1 0 0" />
     </joint>
@@ -93,5 +93,5 @@
         <parent link="${prefix}back_axle" />
         <child link="${prefix}back_left_wheel" />
-        <origin xyz="${-robot_width/2} 0 0" />
+        <origin xyz="${-robot_width/2} 0 -${axle_drop}" />
         <axis xyz="1 0 0" />
     </joint>
