Commit message: Refactor speed handling in CAN hardware to use ros2 control command limits instead of custom logic

File: zoe2_description/urdf/common/params.xacro (robot description, xacro)
@@ -19,3 +19,5 @@
     <xacro:property name="axle_length" value="${robot_width-wheel_thickness}"/>
     <xacro:property name="axle_drop" value="0.119"/>
+    <!-- Speed limits -->
+    <xacro:property name="max_wheel_speed" value="2.0"/>
 </robot>

File: zoe2_description/urdf/zoe2/zoe2_macro.ros2_control.xacro (robot description, xacro)
@@ -42,6 +42,6 @@
           <state_interface name="effort" />
           <command_interface name="velocity" >
-            <param name="min">-10.0</param>
-            <param name="max">10.0</param>
+            <param name="min">-${max_wheel_speed}</param>
+            <param name="max">${max_wheel_speed}</param>
           </command_interface>
       </joint>
@@ -51,6 +51,6 @@
           <state_interface name="effort" />
           <command_interface name="velocity" >
-            <param name="min">-10.0</param>
-            <param name="max">10.0</param>
+            <param name="min">-${max_wheel_speed}</param>
+            <param name="max">${max_wheel_speed}</param>
           </command_interface>
       </joint>
@@ -60,6 +60,6 @@
           <state_interface name="effort" />
           <command_interface name="velocity" >
-            <param name="min">-10.0</param>
-            <param name="max">10.0</param>
+            <param name="min">-${max_wheel_speed}</param>
+            <param name="max">${max_wheel_speed}</param>
           </command_interface>
       </joint>
@@ -69,6 +69,6 @@
           <state_interface name="effort" />
           <command_interface name="velocity" >
-            <param name="min">-10.0</param>
-            <param name="max">10.0</param>
+            <param name="min">-${max_wheel_speed}</param>
+            <param name="max">${max_wheel_speed}</param>
           </command_interface>
       </joint>

Commit message: Adjust proportional gain for zoe2_controller and update max wheel speed parameter

File: zoe2_description/urdf/common/params.xacro (robot description, xacro)
@@ -20,4 +20,4 @@
     <xacro:property name="axle_drop" value="0.119"/>
     <!-- Speed limits -->
-    <xacro:property name="max_wheel_speed" value="2.0"/>
+    <xacro:property name="max_wheel_speed" value="4.0"/>
 </robot>
