Commit message: Re-added {prefix} naming scheme to joints/links for multi-robot support. Note that the rviz is broken, because the links have to be hardcoded to it. This seems inherent to the tools I am using and does not have a simple workaround. I think it should all still function fine outside of rviz, though.

File: zoe2_description/urdf/zoe2/zoe2_macro.ros2_control.xacro (robot description, xacro)
@@ -27,26 +27,26 @@
       </hardware>
       <!-- Joints -->
-      <joint name="front_yaw_joint">
+      <joint name="${prefix}front_yaw_joint">
         <state_interface name="position" />
       </joint>
-      <joint name="back_yaw_joint">
+      <joint name="${prefix}back_yaw_joint">
           <state_interface name="position" />
       </joint>
-      <joint name="front_left_wheel_joint">
+      <joint name="${prefix}front_left_wheel_joint">
           <state_interface name="position" />
           <state_interface name="velocity" />
           <command_interface name="velocity" />
       </joint>
-      <joint name="front_right_wheel_joint">
+      <joint name="${prefix}front_right_wheel_joint">
           <state_interface name="position" />
           <state_interface name="velocity" />
           <command_interface name="velocity" />
       </joint>
-      <joint name="back_right_wheel_joint">
+      <joint name="${prefix}back_right_wheel_joint">
           <state_interface name="position" />
           <state_interface name="velocity" />
           <command_interface name="velocity" />
       </joint>
-      <joint name="back_left_wheel_joint">
+      <joint name="${prefix}back_left_wheel_joint">
           <state_interface name="position" />
           <state_interface name="velocity" />

File: zoe2_description/urdf/zoe2/zoe2_macro.xacro (robot description, xacro)
@@ -10,73 +10,73 @@
   <xacro:macro name="zoe2" params="prefix parent *origin">
     <!-- LINKS -->
-    <link name = "base_link">
+    <link name = "${prefix}base_link">
     </link>
-    <xacro:chassis name="chassis" rpy="0 0 0" xyz="0 0 0" />
-    <xacro:hinge name="front_yaw" rpy="${pi/2} 0 0" xyz="0 0 0" />
-    <xacro:wheel name="front_right_wheel" rpy="0 0 ${pi/2}" xyz="0 0 0" />
-    <xacro:wheel name="front_left_wheel" rpy="0 0 ${-pi/2}" xyz="0 0 0" />
-    <xacro:axle name="front_axle" rpy="${pi/2} 0 0" xyz="0 0 0" />
-    <xacro:wheel name="back_right_wheel" rpy="0 0 ${pi/2}" xyz="0 0 0" />
-    <xacro:wheel name="back_left_wheel" rpy="0 0 ${-pi/2}" xyz="0 0 0" />
-    <xacro:axle name="back_axle" rpy="${pi/2} 0 0" xyz="0 0 0" />
-    <xacro:hinge name="back_yaw" rpy="${-pi/2} 0 0" xyz="0 0 0" />
+    <xacro:chassis name="${prefix}chassis" rpy="0 0 0" xyz="0 0 0" />
+    <xacro:hinge name="${prefix}front_yaw" rpy="${pi/2} 0 0" xyz="0 0 0" />
+    <xacro:wheel name="${prefix}front_right_wheel" rpy="0 0 ${pi/2}" xyz="0 0 0" />
+    <xacro:wheel name="${prefix}front_left_wheel" rpy="0 0 ${-pi/2}" xyz="0 0 0" />
+    <xacro:axle name="${prefix}front_axle" rpy="${pi/2} 0 0" xyz="0 0 0" />
+    <xacro:wheel name="${prefix}back_right_wheel" rpy="0 0 ${pi/2}" xyz="0 0 0" />
+    <xacro:wheel name="${prefix}back_left_wheel" rpy="0 0 ${-pi/2}" xyz="0 0 0" />
+    <xacro:axle name="${prefix}back_axle" rpy="${pi/2} 0 0" xyz="0 0 0" />
+    <xacro:hinge name="${prefix}back_yaw" rpy="${-pi/2} 0 0" xyz="0 0 0" />
     <!-- END LINKS -->
     <!-- JOINTS -->
-    <joint name="base_joint" type="fixed">
+    <joint name="${prefix}base_joint" type="fixed">
         <xacro:insert_block name="origin" />
         <parent link="${parent}" />
-        <child link="base_link" />
+        <child link="${prefix}base_link" />
     </joint>
-    <joint name="chassis_joint" type="fixed">
-        <parent link="base_link" />
-        <child link="chassis" />
+    <joint name="${prefix}chassis_joint" type="fixed">
+        <parent link="${prefix}base_link" />
+        <child link="${prefix}chassis" />
         <origin xyz="0 0 ${wheel_radius}" />
     </joint>
-    <joint name="chassis_front_yaw_joint" type="fixed">
-        <parent link="chassis" />
-        <child link="front_yaw" />
+    <joint name="${prefix}chassis_front_yaw_joint" type="fixed">
+        <parent link="${prefix}chassis" />
+        <child link="${prefix}front_yaw" />
         <origin xyz="0 ${-(robot_length/2 - robot_hinge_length)} 0" />
     </joint>
-    <joint name="front_yaw_joint" type="revolute">
-        <parent link="front_yaw" />
-        <child link="front_axle" />
+    <joint name="${prefix}front_yaw_joint" type="revolute">
+        <parent link="${prefix}front_yaw" />
+        <child link="${prefix}front_axle" />
         <origin xyz="0 ${-robot_hinge_length} -0.075" />
         <axis xyz="0 0 1"/>
         <limit lower="${-front_vertical_limit}" upper="${front_vertical_limit}" effort="0" velocity="0"/>
     </joint>
-    <joint name="front_right_wheel_joint" type="continuous">
-        <parent link="front_axle" />
-        <child link="front_right_wheel" />
+    <joint name="${prefix}front_right_wheel_joint" type="continuous">
+        <parent link="${prefix}front_axle" />
+        <child link="${prefix}front_right_wheel" />
         <origin xyz="${robot_width/2} 0 0" />
         <axis xyz="1 0 0" />
     </joint>
-    <joint name="front_left_wheel_joint" type="continuous">
-        <parent link="front_axle" />
-        <child link="front_left_wheel" />
+    <joint name="${prefix}front_left_wheel_joint" type="continuous">
+        <parent link="${prefix}front_axle" />
+        <child link="${prefix}front_left_wheel" />
         <origin xyz="${-robot_width/2} 0 0" />
         <axis xyz="1 0 0" />
     </joint>
-    <joint name="back_yaw_joint" type="revolute">
-        <parent link="back_yaw" />
-        <child link="back_axle" />
+    <joint name="${prefix}back_yaw_joint" type="revolute">
+        <parent link="${prefix}back_yaw" />
+        <child link="${prefix}back_axle" />
         <origin xyz="0 ${robot_hinge_length} -0.075" />
         <limit lower="${-front_vertical_limit}" upper="${front_vertical_limit}" effort="0" velocity="0"/>
         <axis xyz="0 0 1"/>
     </joint>
-    <joint name="back_right_wheel_joint" type="continuous">
-        <parent link="back_axle" />
-        <child link="back_right_wheel" />
+    <joint name="${prefix}back_right_wheel_joint" type="continuous">
+        <parent link="${prefix}back_axle" />
+        <child link="${prefix}back_right_wheel" />
         <origin xyz="${robot_width/2} 0 0" />
         <axis xyz="1 0 0" />
     </joint>
-    <joint name="back_left_wheel_joint" type="continuous">
-        <parent link="back_axle" />
-        <child link="back_left_wheel" />
+    <joint name="${prefix}back_left_wheel_joint" type="continuous">
+        <parent link="${prefix}back_axle" />
+        <child link="${prefix}back_left_wheel" />
         <origin xyz="${-robot_width/2} 0 0" />
         <axis xyz="1 0 0" />
     </joint>
-    <joint name="chassis_back_yaw_joint" type="fixed">
-        <parent link="chassis" />
-        <child link="back_yaw" />
+    <joint name="${prefix}chassis_back_yaw_joint" type="fixed">
+        <parent link="${prefix}chassis" />
+        <child link="${prefix}back_yaw" />
         <origin xyz="0 ${+(robot_length/2 - robot_hinge_length)} 0" />
     </joint>

Commit message: Readded roll joint

File: zoe2_description/urdf/zoe2/zoe2_macro.ros2_control.xacro (robot description, xacro)
@@ -31,4 +31,7 @@
       </joint>
       <joint name="${prefix}back_yaw_joint">
+          <state_interface name="position" />
+      </joint>
+      <joint name="${prefix}chassis_back_roll_joint">
           <state_interface name="position" />
       </joint>

File: zoe2_description/urdf/zoe2/zoe2_macro.xacro (robot description, xacro)
@@ -13,5 +13,5 @@
     </link>
     <xacro:chassis name="${prefix}chassis" rpy="0 0 0" xyz="0 0 0" />
-    <xacro:hinge name="${prefix}front_yaw" rpy="${pi/2} 0 0" xyz="0 0 0" />
+    <xacro:hinge name="${prefix}front_roll" rpy="${pi/2} 0 0" xyz="0 0 0" />
     <xacro:wheel name="${prefix}front_right_wheel" rpy="0 0 ${pi/2}" xyz="0 0 0" />
     <xacro:wheel name="${prefix}front_left_wheel" rpy="0 0 ${-pi/2}" xyz="0 0 0" />
@@ -20,5 +20,5 @@
     <xacro:wheel name="${prefix}back_left_wheel" rpy="0 0 ${-pi/2}" xyz="0 0 0" />
     <xacro:axle name="${prefix}back_axle" rpy="${pi/2} 0 0" xyz="0 0 0" />
-    <xacro:hinge name="${prefix}back_yaw" rpy="${-pi/2} 0 0" xyz="0 0 0" />
+    <xacro:hinge name="${prefix}back_roll" rpy="${-pi/2} 0 0" xyz="0 0 0" />
     <!-- END LINKS -->
     <!-- JOINTS -->
@@ -33,11 +33,11 @@
         <origin xyz="0 0 ${wheel_radius}" />
     </joint>
-    <joint name="${prefix}chassis_front_yaw_joint" type="fixed">
+    <joint name="${prefix}chassis_front_roll_joint" type="fixed">
         <parent link="${prefix}chassis" />
-        <child link="${prefix}front_yaw" />
+        <child link="${prefix}front_roll" />
         <origin xyz="0 ${-(robot_length/2 - robot_hinge_length)} 0" />
     </joint>
     <joint name="${prefix}front_yaw_joint" type="revolute">
-        <parent link="${prefix}front_yaw" />
+        <parent link="${prefix}front_roll" />
         <child link="${prefix}front_axle" />
         <origin xyz="0 ${-robot_hinge_length} -0.075" />
@@ -58,5 +58,5 @@
     </joint>
     <joint name="${prefix}back_yaw_joint" type="revolute">
-        <parent link="${prefix}back_yaw" />
+        <parent link="${prefix}back_roll" />
         <child link="${prefix}back_axle" />
         <origin xyz="0 ${robot_hinge_length} -0.075" />
@@ -76,8 +76,11 @@
         <axis xyz="1 0 0" />
     </joint>
-    <joint name="${prefix}chassis_back_yaw_joint" type="fixed">
+    <!-- current roll joint limits set arbitrarily... -->
+    <joint name="${prefix}chassis_back_roll_joint" type="revolute">
         <parent link="${prefix}chassis" />
-        <child link="${prefix}back_yaw" />
+        <child link="${prefix}back_roll" />
         <origin xyz="0 ${+(robot_length/2 - robot_hinge_length)} 0" />
+        <limit lower="-0.5" upper="0.5" effort="0" velocity="0"/>
+        <axis xyz="0 1 0" />
     </joint>
     <!-- END JOINTS -->

Commit message: Added basic version of gazebo support. Robot can spawn in, but can't yet be controlled

File: zoe2_description/urdf/zoe2/zoe2_macro.ros2_control.xacro (robot description, xacro)
@@ -6,5 +6,5 @@
                use_mock_hardware:=false
                mock_sensor_commands:=false
-               sim_gazebo_classic:=false
+               sim_gazebo_classic:=true
                sim_gazebo:=false
                simulation_controllers"
@@ -28,30 +28,52 @@
       <!-- Joints -->
       <joint name="${prefix}front_yaw_joint">
-        <state_interface name="position" />
+        <state_interface name="position">
+          <param name="initial_value">0.0</param>
+        </state_interface>
       </joint>
       <joint name="${prefix}back_yaw_joint">
-          <state_interface name="position" />
+          <state_interface name="position">
+            <param name="initial_value">0.0</param>
+          </state_interface>
       </joint>
       <joint name="${prefix}chassis_back_roll_joint">
-          <state_interface name="position" />
+          <state_interface name="position">
+            <param name="initial_value">0.0</param>
+          </state_interface>
       </joint>
       <joint name="${prefix}front_left_wheel_joint">
-          <state_interface name="position" />
-          <state_interface name="velocity" />
+          <state_interface name="position">
+            <param name="initial_value">0.0</param>
+          </state_interface>
+          <state_interface name="velocity">
+            <param name="initial_value">0.0</param>
+          </state_interface>
           <command_interface name="velocity" />
       </joint>
       <joint name="${prefix}front_right_wheel_joint">
-          <state_interface name="position" />
-          <state_interface name="velocity" />
+          <state_interface name="position">
+            <param name="initial_value">0.0</param>
+          </state_interface>
+          <state_interface name="velocity">
+            <param name="initial_value">0.0</param>
+          </state_interface>
           <command_interface name="velocity" />
       </joint>
       <joint name="${prefix}back_right_wheel_joint">
-          <state_interface name="position" />
-          <state_interface name="velocity" />
+          <state_interface name="position">
+            <param name="initial_value">0.0</param>
+          </state_interface>
+          <state_interface name="velocity">
+            <param name="initial_value">0.0</param>
+          </state_interface>
           <command_interface name="velocity" />
       </joint>
       <joint name="${prefix}back_left_wheel_joint">
-          <state_interface name="position" />
-          <state_interface name="velocity" />
+          <state_interface name="position">
+            <param name="initial_value">0.0</param>
+          </state_interface>
+          <state_interface name="velocity">
+            <param name="initial_value">0.0</param>
+          </state_interface>
           <command_interface name="velocity" />
       </joint>

File: zoe2_description/urdf/zoe2/zoe2_macro.xacro (robot description, xacro)
@@ -43,5 +43,5 @@
         <origin xyz="0 ${-robot_hinge_length} -0.075" />
         <axis xyz="0 0 1"/>
-        <limit lower="${-front_vertical_limit}" upper="${front_vertical_limit}" effort="0" velocity="0"/>
+        <limit lower="${-front_vertical_limit}" upper="${front_vertical_limit}" effort="10" velocity="10"/>
     </joint>
     <joint name="${prefix}front_right_wheel_joint" type="continuous">
@@ -61,5 +61,5 @@
         <child link="${prefix}back_axle" />
         <origin xyz="0 ${robot_hinge_length} -0.075" />
-        <limit lower="${-front_vertical_limit}" upper="${front_vertical_limit}" effort="0" velocity="0"/>
+        <limit lower="${-front_vertical_limit}" upper="${front_vertical_limit}" effort="10" velocity="10"/>
         <axis xyz="0 0 1"/>
     </joint>
@@ -81,5 +81,5 @@
         <child link="${prefix}back_roll" />
         <origin xyz="0 ${+(robot_length/2 - robot_hinge_length)} 0" />
-        <limit lower="-0.5" upper="0.5" effort="0" velocity="0"/>
+        <limit lower="-0.5" upper="0.5" effort="10" velocity="10"/>
         <axis xyz="0 1 0" />
     </joint>

Commit message: Corrected issue in launch file and re-enable yaw joint mobility

File: zoe2_description/urdf/zoe2/zoe2_macro.ros2_control.xacro (robot description, xacro)
@@ -27,10 +27,10 @@
       </hardware>
       <!-- Pivot Joints -->
-      <!-- <joint name="${prefix}front_yaw_joint">
+      <joint name="${prefix}front_yaw_joint">
         <state_interface name="position" />
       </joint>
       <joint name="${prefix}back_yaw_joint">
           <state_interface name="position" />
-      </joint> -->
+      </joint>
       <joint name="${prefix}chassis_back_roll_joint">
           <state_interface name="position" />

File: zoe2_description/urdf/zoe2/zoe2_macro.xacro (robot description, xacro)
@@ -35,11 +35,10 @@
         <origin xyz="0 ${-(robot_length/2 - robot_hinge_length)} 0" />
     </joint>
-    <!-- temp set to fixed -->
-    <joint name="${prefix}front_yaw_joint" type="fixed">
+    <joint name="${prefix}front_yaw_joint" type="revolute">
         <parent link="${prefix}front_roll" />
         <child link="${prefix}front_axle" />
         <origin xyz="0 ${-robot_hinge_length} -0.075" />
-        <!-- <axis xyz="0 0 1"/>
-        <limit lower="${-front_vertical_limit}" upper="${front_vertical_limit}" effort="10" velocity="10"/> -->
+        <axis xyz="0 0 1"/>
+        <limit lower="${-front_vertical_limit}" upper="${front_vertical_limit}" effort="10" velocity="10"/>
     </joint>
     <joint name="${prefix}front_right_wheel_joint" type="continuous">
@@ -56,10 +55,10 @@
     </joint>
     <!-- temp set to fixed -->
-    <joint name="${prefix}back_yaw_joint" type="fixed">
+    <joint name="${prefix}back_yaw_joint" type="revolute">
         <parent link="${prefix}back_roll" />
         <child link="${prefix}back_axle" />
         <origin xyz="0 ${robot_hinge_length} -0.075" />
-        <!-- <limit lower="${-front_vertical_limit}" upper="${front_vertical_limit}" effort="10" velocity="10"/>
-        <axis xyz="0 0 1"/> -->
+        <limit lower="${-front_vertical_limit}" upper="${front_vertical_limit}" effort="10" velocity="10"/>
+        <axis xyz="0 0 1"/>
     </joint>
     <joint name="${prefix}back_right_wheel_joint" type="continuous">

Commit message: Change roll axle to front; update speed clamping logic

File: zoe2_description/urdf/zoe2/zoe2_macro.ros2_control.xacro (robot description, xacro)
@@ -33,5 +33,5 @@
           <state_interface name="position" />
       </joint>
-      <joint name="${prefix}axle_roll_back_joint">
+      <joint name="${prefix}axle_roll_front_joint">
           <state_interface name="position" />
       </joint>

File: zoe2_description/urdf/zoe2/zoe2_macro.xacro (robot description, xacro)
@@ -52,8 +52,10 @@
         <origin xyz="0 0 ${base_link_height}" />
     </joint>
-    <joint name="${prefix}chassis_front_roll_joint" type="fixed">
+    <joint name="${prefix}axle_roll_front_joint" type="revolute">
         <parent link="${prefix}chassis" />
         <child link="${prefix}front_roll" />
         <origin xyz="0 ${(robot_length/2 - robot_hinge_length)} 0" />
+        <limit lower="-0.5" upper="0.5" effort="10" velocity="10"/>
+        <axis xyz="0 1 0" />
     </joint>
     <joint name="${prefix}axle_yaw_front_joint" type="revolute">
@@ -97,10 +99,8 @@
     </joint>
     <!-- current roll joint limits set arbitrarily... -->
-    <joint name="${prefix}axle_roll_back_joint" type="revolute">
+    <joint name="${prefix}axle_roll_back_joint" type="fixed">
         <parent link="${prefix}chassis" />
         <child link="${prefix}back_roll" />
         <origin xyz="0 ${-(robot_length/2 - robot_hinge_length)} 0" />
-        <limit lower="-0.5" upper="0.5" effort="10" velocity="10"/>
-        <axis xyz="0 1 0" />
     </joint>
     <!-- END JOINTS -->
