Commit message: Added moon world

File: zoe2_description/urdf/zoe2/zoe2_macro.xacro (robot description, xacro)
@@ -23,4 +23,26 @@
     <xacro:axle name="${prefix}back_axle" rpy="${pi/2} 0 0" xyz="0 0 0" />
     <xacro:hinge name="${prefix}back_roll" rpy="${-pi/2} 0 0" xyz="0 0 0" />
+    <!-- Link gazebo params -->
+    <gazebo reference="back_left_wheel">
+        <material>Gazebo/Black</material>
+    </gazebo>
+    <gazebo reference="back_right_wheel">
+        <material>Gazebo/Black</material>
+    </gazebo>
+    <gazebo reference="front_right_wheel">
+        <material>Gazebo/Black</material>
+    </gazebo>
+    <gazebo reference="front_left_wheel">
+        <material>Gazebo/Black</material>
+    </gazebo>
+    <gazebo reference="chassis">
+        <material>Gazebo/Blue</material>
+    </gazebo>
+    <gazebo reference="front_axle">
+        <material>Gazebo/Blue</material>
+    </gazebo>
+    <gazebo reference="back_axle">
+        <material>Gazebo/Blue</material>
+    </gazebo>
     <!-- END LINKS -->
     <!-- JOINTS -->

Commit message: Fix joint origin and axis configurations in URDF; update error calculations in controller

File: zoe2_description/urdf/zoe2/zoe2_macro.xacro (robot description, xacro)
@@ -55,10 +55,10 @@
         <parent link="${prefix}chassis" />
         <child link="${prefix}front_roll" />
-        <origin xyz="0 ${-(robot_length/2 - robot_hinge_length)} 0" />
+        <origin xyz="0 ${(robot_length/2 - robot_hinge_length)} 0" />
     </joint>
     <joint name="${prefix}front_yaw_joint" type="revolute">
         <parent link="${prefix}front_roll" />
         <child link="${prefix}front_axle" />
-        <origin xyz="0 ${-robot_hinge_length} 0" />
+        <origin xyz="0 ${robot_hinge_length} 0" />
         <axis xyz="0 0 1"/>
         <limit lower="${-front_vertical_limit}" upper="${front_vertical_limit}" effort="10" velocity="10"/>
@@ -68,5 +68,5 @@
         <child link="${prefix}front_right_wheel" />
         <origin xyz="${robot_width/2} 0 -${axle_drop}" />
-        <axis xyz="1 0 0" />
+        <axis xyz="-1 0 0" />
     </joint>
     <joint name="${prefix}front_left_wheel_joint" type="continuous">
@@ -74,5 +74,5 @@
         <child link="${prefix}front_left_wheel" />
         <origin xyz="${-robot_width/2} 0 -${axle_drop}" />
-        <axis xyz="1 0 0" />
+        <axis xyz="-1 0 0" />
     </joint>
     <!-- temp set to fixed -->
@@ -80,5 +80,5 @@
         <parent link="${prefix}back_roll" />
         <child link="${prefix}back_axle" />
-        <origin xyz="0 ${robot_hinge_length} 0" />
+        <origin xyz="0 ${-robot_hinge_length} 0" />
         <limit lower="${-front_vertical_limit}" upper="${front_vertical_limit}" effort="10" velocity="10"/>
         <axis xyz="0 0 1"/>
@@ -88,5 +88,5 @@
         <child link="${prefix}back_right_wheel" />
         <origin xyz="${robot_width/2} 0 -${axle_drop}" />
-        <axis xyz="1 0 0" />
+        <axis xyz="-1 0 0" />
     </joint>
     <joint name="${prefix}back_left_wheel_joint" type="continuous">
@@ -94,5 +94,5 @@
         <child link="${prefix}back_left_wheel" />
         <origin xyz="${-robot_width/2} 0 -${axle_drop}" />
-        <axis xyz="1 0 0" />
+        <axis xyz="-1 0 0" />
     </joint>
     <!-- current roll joint limits set arbitrarily... -->
@@ -100,5 +100,5 @@
         <parent link="${prefix}chassis" />
         <child link="${prefix}back_roll" />
-        <origin xyz="0 ${+(robot_length/2 - robot_hinge_length)} 0" />
+        <origin xyz="0 ${-(robot_length/2 - robot_hinge_length)} 0" />
         <limit lower="-0.5" upper="0.5" effort="10" velocity="10"/>
         <axis xyz="0 1 0" />

Commit message: Add antenna part and parameters to Zoe2 URDF model

File: zoe2_description/urdf/zoe2/zoe2_macro.xacro (robot description, xacro)
@@ -9,4 +9,5 @@
   <xacro:include filename="$(find zoe2_description)/urdf/zoe2/parts/axle.xacro" />
   <xacro:include filename="$(find zoe2_description)/urdf/zoe2/parts/hinge.xacro" />
+  <xacro:include filename="$(find zoe2_description)/urdf/zoe2/parts/antenna.xacro" />
   <xacro:include filename="$(find zoe2_description)/urdf/zoe2/zoe2_params.xacro" />
   <xacro:macro name="zoe2" params="prefix *origin">
@@ -23,4 +24,5 @@
     <xacro:axle name="${prefix}back_axle" rpy="${pi/2} 0 ${pi/2}" xyz="0 0 0" />
     <xacro:hinge name="${prefix}back_roll" rpy="${-pi/2} 0 0" xyz="0 0 0" />
+    <xacro:antenna name="${prefix}antenna" rpy="0 0 0" xyz="0 0 ${antenna_length/2}" />
     <!-- Link gazebo params -->
     <gazebo reference="wheel_back_left">
@@ -52,4 +54,9 @@
         <origin xyz="0 0 ${base_link_height}" />
     </joint>
+    <joint name="${prefix}antenna_joint" type="fixed">
+        <parent link="${prefix}chassis" />
+        <child link="${prefix}antenna" />
+        <origin xyz="0 ${antenna_location} ${chassis_height}" />
+    </joint>
     <joint name="${prefix}axle_roll_front_joint" type="revolute">
         <parent link="${prefix}chassis" />
@@ -78,5 +85,4 @@
         <axis xyz="-1 0 0" />
     </joint>
-    <!-- temp set to fixed -->
     <joint name="${prefix}axle_yaw_back_joint" type="revolute">
         <parent link="${prefix}back_roll" />
@@ -98,5 +104,4 @@
         <axis xyz="-1 0 0" />
     </joint>
-    <!-- current roll joint limits set arbitrarily... -->
     <joint name="${prefix}axle_roll_back_joint" type="fixed">
         <parent link="${prefix}chassis" />

File: zoe2_description/urdf/zoe2/zoe2_params.xacro (robot description, xacro)
@@ -19,4 +19,8 @@
     <xacro:property name="axle_length" value="${robot_width-wheel_thickness}"/>
     <xacro:property name="axle_drop" value="0"/>
+    <!-- Antenna -->
+    <xacro:property name="antenna_length" value="0.52"/>
+    <xacro:property name="antenna_radius" value="0.015"/>
+    <xacro:property name="antenna_location" value="-0.3"/>
     <!-- Speed limits -->
     <xacro:property name="max_wheel_speed" value="4.0"/>
