Commit message: Fix base width parameter in zoe2 controller and URDF

File: zoe2_description/urdf/zoe2/zoe2_params.xacro (robot description, xacro)
@@ -2,5 +2,5 @@
     <robot xmlns:xacro="http://www.ros.org/wiki/xacro"  name="robot">
     <!-- all are in meters -->
-    <xacro:property name="robot_width" value="1.115" />
+    <xacro:property name="robot_width" value="1.1115" />
     <xacro:property name="robot_length" value="1.264"/>
     <xacro:property name="base_link_height" value="0.2"/>
