Commit message: Update urdf params and layout to match Zoe2

File: zoe2_description/urdf/zoe2/parts/chassis.xacro (robot description, xacro)
@@ -34,5 +34,5 @@
             <collision>
                 <origin
-                    xyz="0 0 ${chassis_height/2-axle_box_width/2}"
+                    xyz="0 0 ${chassis_height/2}"
                     rpy="${rpy}" />
                 <geometry>

File: zoe2_description/urdf/zoe2/zoe2_macro.xacro (robot description, xacro)
@@ -55,5 +55,5 @@
         <parent link="${prefix}chassis" />
         <child link="${prefix}front_roll" />
-        <origin xyz="0 ${(robot_length/2 - robot_hinge_length)} 0" />
+        <origin xyz="0 ${(robot_length/2 - robot_hinge_length)} ${wheel_radius-base_link_height}" />
         <limit lower="-0.5" upper="0.5" effort="10" velocity="10"/>
         <axis xyz="0 1 0" />
@@ -102,5 +102,5 @@
         <parent link="${prefix}chassis" />
         <child link="${prefix}back_roll" />
-        <origin xyz="0 ${-(robot_length/2 - robot_hinge_length)} 0" />
+        <origin xyz="0 ${-(robot_length/2 - robot_hinge_length)} ${wheel_radius-base_link_height}" />
     </joint>
     <!-- END JOINTS -->

File: zoe2_description/urdf/zoe2/zoe2_params.xacro (robot description, xacro)
@@ -2,21 +2,21 @@
     <robot xmlns:xacro="http://www.ros.org/wiki/xacro"  name="robot">
     <!-- all are in meters -->
-    <xacro:property name="robot_width" value="1.64" />
-    <xacro:property name="robot_length" value="1.91"/>
-    <xacro:property name="base_link_height" value="0.4"/>
+    <xacro:property name="robot_width" value="1.115" />
+    <xacro:property name="robot_length" value="1.264"/>
+    <xacro:property name="base_link_height" value="0.2"/>
     <!-- Chassis -->
-    <xacro:property name="chassis_length" value="1.5"/>
-    <xacro:property name="chassis_width" value="1.2"/>
-    <xacro:property name="chassis_height" value="0.5"/>
+    <xacro:property name="chassis_length" value="1"/>
+    <xacro:property name="chassis_width" value="0.230"/>
+    <xacro:property name="chassis_height" value="0.3"/>
     <!-- Hinge -->
-    <xacro:property name="robot_hinge_length" value="0.2"/>
+    <xacro:property name="robot_hinge_length" value="0.132"/>
     <xacro:property name="front_vertical_limit" value="${pi/4}"/>
     <!-- Wheel -->
-    <xacro:property name="wheel_radius" value="0.325"/>
-    <xacro:property name="wheel_thickness" value="0.05"/>
+    <xacro:property name="wheel_radius" value="0.292"/>
+    <xacro:property name="wheel_thickness" value="0.074"/>
     <!-- Axle -->
     <xacro:property name="axle_box_width" value="0.1"/>
     <xacro:property name="axle_length" value="${robot_width-wheel_thickness}"/>
-    <xacro:property name="axle_drop" value="0.119"/>
+    <xacro:property name="axle_drop" value="0"/>
     <!-- Speed limits -->
     <xacro:property name="max_wheel_speed" value="4.0"/>
