Commit message: Update zoe2 urdf to use cylindrical axle

File: zoe2_description/urdf/zoe2/parts/axle.xacro (robot description, xacro)
@@ -39,5 +39,5 @@
                     <!-- <mesh
                         filename="file://$(find zoe2_description)/meshes/zoe2/collision/front_axle.STL" /> -->
-                    <box size="${axle_length} ${axle_box_width} ${axle_box_width}" />
+                    <cylinder length="${axle_length}" radius="${axle_radius}" />
                 </geometry>
             </collision>

File: zoe2_description/urdf/zoe2/parts/hinge.xacro (robot description, xacro)
@@ -39,5 +39,5 @@
                     <!-- <mesh
                         filename="file://$(find zoe2_description)/meshes/zoe2/collision/back_hinge.STL" /> -->
-                    <box size="${axle_box_width} ${axle_box_width} ${robot_hinge_length*2}" />
+                    <box size="${axle_radius} ${axle_radius} ${robot_hinge_length*2}" />
                 </geometry>
             </collision>

File: zoe2_description/urdf/zoe2/zoe2_macro.xacro (robot description, xacro)
@@ -18,8 +18,8 @@
     <xacro:wheel name="${prefix}wheel_front_right" rpy="0 0 ${pi/2}" xyz="0 0 0" />
     <xacro:wheel name="${prefix}wheel_front_left" rpy="0 0 ${-pi/2}" xyz="0 0 0" />
-    <xacro:axle name="${prefix}front_axle" rpy="${pi/2} 0 0" xyz="0 0 0" />
+    <xacro:axle name="${prefix}front_axle" rpy="${pi/2} 0 ${pi/2}" xyz="0 0 0" />
     <xacro:wheel name="${prefix}wheel_back_right" rpy="0 0 ${pi/2}" xyz="0 0 0" />
     <xacro:wheel name="${prefix}wheel_back_left" rpy="0 0 ${-pi/2}" xyz="0 0 0" />
-    <xacro:axle name="${prefix}back_axle" rpy="${pi/2} 0 0" xyz="0 0 0" />
+    <xacro:axle name="${prefix}back_axle" rpy="${pi/2} 0 ${pi/2}" xyz="0 0 0" />
     <xacro:hinge name="${prefix}back_roll" rpy="${-pi/2} 0 0" xyz="0 0 0" />
     <!-- Link gazebo params -->

File: zoe2_description/urdf/zoe2/zoe2_params.xacro (robot description, xacro)
@@ -16,5 +16,5 @@
     <xacro:property name="wheel_thickness" value="0.074"/>
     <!-- Axle -->
-    <xacro:property name="axle_box_width" value="0.1"/>
+    <xacro:property name="axle_radius" value="0.05715"/>
     <xacro:property name="axle_length" value="${robot_width-wheel_thickness}"/>
     <xacro:property name="axle_drop" value="0"/>
