Commit message: Refactor URDF components to replace zoe1 mesh geometries with primitive shapes for antenna, axle, chassis, hinge, and wheel parts until proper meshes are added

File: zoe2_description/urdf/zoe2/parts/antenna.xacro (robot description, xacro)
@@ -12,4 +12,17 @@
                 </geometry>
             </collision>
+            <visual>
+                <origin
+                    xyz="${xyz}"
+                    rpy="${rpy}" />
+                <geometry>
+                    <cylinder length="${antenna_length}" radius="${antenna_radius}" />
+                </geometry>
+                <material
+                    name="">
+                    <color
+                        rgba="0.866666666666667 0.909803921568627 1 1" />
+                </material>
+            </visual>
         </link>
     </xacro:macro>

File: zoe2_description/urdf/zoe2/parts/axle.xacro (robot description, xacro)
@@ -23,6 +23,7 @@
                     rpy="${rpy}" />
                 <geometry>
-                    <mesh
-                        filename="file://$(find zoe2_description)/meshes/zoe2/collision/front_axle.STL" />
+                    <!-- <mesh
+                        filename="file://$(find zoe2_description)/meshes/zoe2/collision/front_axle.STL" /> -->
+                    <cylinder length="${axle_length}" radius="${axle_radius}" />
                 </geometry>
                 <material

File: zoe2_description/urdf/zoe2/parts/chassis.xacro (robot description, xacro)
@@ -23,6 +23,7 @@
                     rpy="${rpy}" />
                 <geometry>
-                    <mesh
-                        filename="file://$(find zoe2_description)/meshes/zoe2/collision/chassis.STL" />
+                    <!-- <mesh
+                        filename="file://$(find zoe2_description)/meshes/zoe2/collision/chassis.STL" /> -->
+                    <box size="${chassis_width} ${chassis_length} ${chassis_height}" />
                 </geometry>
                 <material
@@ -34,5 +35,5 @@
             <collision>
                 <origin
-                    xyz="0 0 ${chassis_height/2}"
+                    xyz="${xyz}"
                     rpy="${rpy}" />
                 <geometry>

File: zoe2_description/urdf/zoe2/parts/hinge.xacro (robot description, xacro)
@@ -23,6 +23,7 @@
                     rpy="${rpy}" />
                 <geometry>
-                    <mesh
-                        filename="file://$(find zoe2_description)/meshes/zoe2/collision/back_hinge.STL" />
+                    <!-- <mesh
+                        filename="file://$(find zoe2_description)/meshes/zoe2/collision/back_hinge.STL" /> -->
+                    <box size="${axle_radius} ${axle_radius} ${robot_hinge_length*2}" />
                 </geometry>
                 <material

File: zoe2_description/urdf/zoe2/parts/wheel.xacro (robot description, xacro)
@@ -23,6 +23,7 @@
                     rpy="${rpy}" />
                 <geometry>
-                    <mesh
-                        filename="file://$(find zoe2_description)/meshes/zoe2/collision/wheel_back_right.STL" />
+                    <!-- <mesh
+                        filename="file://$(find zoe2_description)/meshes/zoe2/collision/wheel_back_right.STL" /> -->
+                  <cylinder radius="${wheel_radius}" length="${wheel_thickness}"/>
                 </geometry>
                 <material
@@ -35,5 +36,5 @@
                 <origin
                     xyz="${xyz}"
-                    rpy="0 ${-pi/2} 0" />
+                    rpy="${rpy}" />
                 <geometry>
                     <!-- <mesh

File: zoe2_description/urdf/zoe2/zoe2_macro.xacro (robot description, xacro)
@@ -15,11 +15,11 @@
     <link name = "${prefix}base_link">
     </link>
-    <xacro:chassis name="${prefix}chassis" rpy="0 0 0" xyz="0 0 0" />
+    <xacro:chassis name="${prefix}chassis" rpy="0 0 0" xyz="0 0 ${chassis_height/2}" />
     <xacro:hinge name="${prefix}front_roll" rpy="${pi/2} 0 0" xyz="0 0 0" />
-    <xacro:wheel name="${prefix}wheel_front_right" rpy="0 0 ${pi/2}" xyz="0 0 0" />
-    <xacro:wheel name="${prefix}wheel_front_left" rpy="0 0 ${-pi/2}" xyz="0 0 0" />
+    <xacro:wheel name="${prefix}wheel_front_right" rpy="0 ${pi/2} 0" xyz="0 0 0" />
+    <xacro:wheel name="${prefix}wheel_front_left" rpy="0 ${-pi/2} 0" xyz="0 0 0" />
     <xacro:axle name="${prefix}front_axle" rpy="${pi/2} 0 ${pi/2}" xyz="0 0 0" />
-    <xacro:wheel name="${prefix}wheel_back_right" rpy="0 0 ${pi/2}" xyz="0 0 0" />
-    <xacro:wheel name="${prefix}wheel_back_left" rpy="0 0 ${-pi/2}" xyz="0 0 0" />
+    <xacro:wheel name="${prefix}wheel_back_right" rpy="0 ${pi/2} 0" xyz="0 0 0" />
+    <xacro:wheel name="${prefix}wheel_back_left" rpy="0 ${-pi/2} 0" xyz="0 0 0" />
     <xacro:axle name="${prefix}back_axle" rpy="${pi/2} 0 ${pi/2}" xyz="0 0 0" />
     <xacro:hinge name="${prefix}back_roll" rpy="${-pi/2} 0 0" xyz="0 0 0" />
