Commit message: Fixed Zoe2 being fixed to the world. Can now move freely.

File: zoe2_description/urdf/zoe2.urdf.xacro (robot description, xacro)
@@ -10,9 +10,7 @@
   <xacro:include filename="$(find zoe2_description)/urdf/zoe2/zoe2_macro.xacro"/>
   <xacro:include filename="$(find zoe2_description)/urdf/zoe2/zoe2_macro.ros2_control.xacro"/>
-  <!-- create link fixed to the "world" -->
-  <link name="world" />
   <!-- Load robot's macro with parameters -->
   <!-- set prefix if multiple robots are used -->
-  <xacro:zoe2 prefix="$(arg prefix)" parent="world" >
+  <xacro:zoe2 prefix="$(arg prefix)" >
     <origin xyz="0 0 0" rpy="0 0 0" />          <!-- position robot in the world -->
   </xacro:zoe2>

File: zoe2_description/urdf/zoe2/zoe2_macro.xacro (robot description, xacro)
@@ -8,5 +8,5 @@
   <xacro:include filename="$(find zoe2_description)/urdf/common/hinge.xacro" />
   <xacro:include filename="$(find zoe2_description)/urdf/common/params.xacro" />
-  <xacro:macro name="zoe2" params="prefix parent *origin">
+  <xacro:macro name="zoe2" params="prefix *origin">
     <!-- LINKS -->
     <link name = "${prefix}base_link">
@@ -23,9 +23,4 @@
     <!-- END LINKS -->
     <!-- JOINTS -->
-    <joint name="${prefix}base_joint" type="fixed">
-        <xacro:insert_block name="origin" />
-        <parent link="${parent}" />
-        <child link="${prefix}base_link" />
-    </joint>
     <joint name="${prefix}chassis_joint" type="fixed">
         <parent link="${prefix}base_link" />

Commit message: Initial Diff Drive functionality, robot is able to spawn and drive around

File: zoe2_description/urdf/zoe2.urdf.xacro (robot description, xacro)
@@ -5,7 +5,7 @@
   <xacro:arg name="use_mock_hardware" default="false" />
   <xacro:arg name="mock_sensor_commands" default="false" />
-  <xacro:arg name="sim_gazebo_classic" default="false" />
+  <xacro:arg name="sim_gazebo_classic" default="true" />
   <xacro:arg name="sim_gazebo" default="false" />
-  <xacro:arg name="simulation_controllers" default="" />
+  <xacro:arg name="simulation_controllers" default="$(find zoe2_bringup)/config/zoe2_controllers.yaml" />
   <xacro:include filename="$(find zoe2_description)/urdf/zoe2/zoe2_macro.xacro"/>
   <xacro:include filename="$(find zoe2_description)/urdf/zoe2/zoe2_macro.ros2_control.xacro"/>
@@ -13,4 +13,5 @@
   <!-- set prefix if multiple robots are used -->
   <xacro:zoe2 prefix="$(arg prefix)" >
+    <!-- TODO: Check if origin is actually implemented -->
     <origin xyz="0 0 0" rpy="0 0 0" />          <!-- position robot in the world -->
   </xacro:zoe2>

File: zoe2_description/urdf/zoe2/zoe2_macro.ros2_control.xacro (robot description, xacro)
@@ -6,5 +6,5 @@
                use_mock_hardware:=false
                mock_sensor_commands:=false
-               sim_gazebo_classic:=true
+               sim_gazebo_classic:=false
                sim_gazebo:=false
                simulation_controllers"
@@ -26,55 +26,46 @@
         </xacro:unless>
       </hardware>
-      <!-- Joints -->
-      <joint name="${prefix}front_yaw_joint">
-        <state_interface name="position">
-          <param name="initial_value">0.0</param>
-        </state_interface>
+      <!-- Pivot Joints -->
+      <!-- <joint name="${prefix}front_yaw_joint">
+        <state_interface name="position" />
       </joint>
       <joint name="${prefix}back_yaw_joint">
-          <state_interface name="position">
-            <param name="initial_value">0.0</param>
-          </state_interface>
+          <state_interface name="position" />
+      </joint> -->
+      <joint name="${prefix}chassis_back_roll_joint">
+          <state_interface name="position" />
       </joint>
-      <joint name="${prefix}chassis_back_roll_joint">
-          <state_interface name="position">
-            <param name="initial_value">0.0</param>
-          </state_interface>
-      </joint>
+      <!-- Wheel Joints -->
       <joint name="${prefix}front_left_wheel_joint">
-          <state_interface name="position">
-            <param name="initial_value">0.0</param>
-          </state_interface>
-          <state_interface name="velocity">
-            <param name="initial_value">0.0</param>
-          </state_interface>
-          <command_interface name="velocity" />
+          <state_interface name="position" />
+          <state_interface name="velocity" />
+          <command_interface name="velocity" >
+            <param name="min">-10.0</param>
+            <param name="max">10.0</param>
+          </command_interface>
       </joint>
       <joint name="${prefix}front_right_wheel_joint">
-          <state_interface name="position">
-            <param name="initial_value">0.0</param>
-          </state_interface>
-          <state_interface name="velocity">
-            <param name="initial_value">0.0</param>
-          </state_interface>
-          <command_interface name="velocity" />
+          <state_interface name="position" />
+          <state_interface name="velocity" />
+          <command_interface name="velocity" >
+            <param name="min">-10.0</param>
+            <param name="max">10.0</param>
+          </command_interface>
       </joint>
       <joint name="${prefix}back_right_wheel_joint">
-          <state_interface name="position">
-            <param name="initial_value">0.0</param>
-          </state_interface>
-          <state_interface name="velocity">
-            <param name="initial_value">0.0</param>
-          </state_interface>
-          <command_interface name="velocity" />
+          <state_interface name="position" />
+          <state_interface name="velocity" />
+          <command_interface name="velocity" >
+            <param name="min">-10.0</param>
+            <param name="max">10.0</param>
+          </command_interface>
       </joint>
       <joint name="${prefix}back_left_wheel_joint">
-          <state_interface name="position">
-            <param name="initial_value">0.0</param>
-          </state_interface>
-          <state_interface name="velocity">
-            <param name="initial_value">0.0</param>
-          </state_interface>
-          <command_interface name="velocity" />
+          <state_interface name="position" />
+          <state_interface name="velocity" />
+          <command_interface name="velocity" >
+            <param name="min">-10.0</param>
+            <param name="max">10.0</param>
+          </command_interface>
       </joint>
     </ros2_control>

File: zoe2_description/urdf/zoe2/zoe2_macro.xacro (robot description, xacro)
@@ -1,3 +1,5 @@
 <?xml version="1.0" encoding="UTF-8"?>
+<!-- This macro defines the actual link-joint structure of the robot. -->
+<!-- The macro can be called by other files via <xacro:zoe2 prefix="$(arg prefix)" > -->
 <robot xmlns:xacro="http://wiki.ros.org/xacro">
   <xacro:include filename="$(find zoe2_description)/urdf/common/inertials.xacro" />
@@ -33,10 +35,11 @@
         <origin xyz="0 ${-(robot_length/2 - robot_hinge_length)} 0" />
     </joint>
-    <joint name="${prefix}front_yaw_joint" type="revolute">
+    <!-- temp set to fixed -->
+    <joint name="${prefix}front_yaw_joint" type="fixed">
         <parent link="${prefix}front_roll" />
         <child link="${prefix}front_axle" />
         <origin xyz="0 ${-robot_hinge_length} -0.075" />
-        <axis xyz="0 0 1"/>
-        <limit lower="${-front_vertical_limit}" upper="${front_vertical_limit}" effort="10" velocity="10"/>
+        <!-- <axis xyz="0 0 1"/>
+        <limit lower="${-front_vertical_limit}" upper="${front_vertical_limit}" effort="10" velocity="10"/> -->
     </joint>
     <joint name="${prefix}front_right_wheel_joint" type="continuous">
@@ -52,10 +55,11 @@
         <axis xyz="1 0 0" />
     </joint>
-    <joint name="${prefix}back_yaw_joint" type="revolute">
+    <!-- temp set to fixed -->
+    <joint name="${prefix}back_yaw_joint" type="fixed">
         <parent link="${prefix}back_roll" />
         <child link="${prefix}back_axle" />
         <origin xyz="0 ${robot_hinge_length} -0.075" />
-        <limit lower="${-front_vertical_limit}" upper="${front_vertical_limit}" effort="10" velocity="10"/>
-        <axis xyz="0 0 1"/>
+        <!-- <limit lower="${-front_vertical_limit}" upper="${front_vertical_limit}" effort="10" velocity="10"/>
+        <axis xyz="0 0 1"/> -->
     </joint>
     <joint name="${prefix}back_right_wheel_joint" type="continuous">

Commit message: Add locking parameters for front and back yaw and roll joints in URDF macros

File: zoe2_description/urdf/zoe2.urdf.xacro (robot description, xacro)
@@ -8,12 +8,16 @@
   <xacro:arg name="sim_gazebo" default="false" />
   <xacro:arg name="simulation_controllers" default="$(find zoe2_bringup)/config/zoe2_sim_controllers.yaml" />
+  <xacro:arg name="lock_front_yaw" default="false" />
+  <xacro:arg name="lock_front_roll" default="false" />
+  <xacro:arg name="lock_back_yaw" default="false" />
   <xacro:include filename="$(find zoe2_description)/urdf/zoe2/zoe2_macro.xacro"/>
   <xacro:include filename="$(find zoe2_description)/urdf/zoe2/zoe2_macro.ros2_control.xacro"/>
   <!-- Load robot's macro with parameters -->
   <!-- set prefix if multiple robots are used -->
-  <xacro:zoe2 prefix="$(arg prefix)" >
-    <!-- TODO: Check if origin is actually implemented -->
-    <origin xyz="0 0 0" rpy="0 0 0" />          <!-- position robot in the world -->
-  </xacro:zoe2>
+  <xacro:zoe2 prefix="$(arg prefix)"
+    lock_front_yaw="$(arg lock_front_yaw)"
+    lock_front_roll="$(arg lock_front_roll)"
+    lock_back_yaw="$(arg lock_back_yaw)"
+  />
   <xacro:zoe2_ros2_control
     name="zoe2"
@@ -23,4 +27,8 @@
     sim_gazebo_classic="$(arg sim_gazebo_classic)"
     sim_gazebo="$(arg sim_gazebo)"
-    simulation_controllers="$(arg simulation_controllers)" />
+    simulation_controllers="$(arg simulation_controllers)"
+    lock_front_yaw="$(arg lock_front_yaw)"
+    lock_front_roll="$(arg lock_front_roll)"
+    lock_back_yaw="$(arg lock_back_yaw)"
+    />
 </robot>

File: zoe2_description/urdf/zoe2/zoe2_macro.ros2_control.xacro (robot description, xacro)
@@ -8,6 +8,9 @@
                sim_gazebo_classic:=false
                sim_gazebo:=false
-               simulation_controllers"
-               >
+               simulation_controllers
+               lock_front_yaw:=true
+               lock_front_roll:=false
+               lock_back_yaw:=false
+               ">
     <ros2_control name="${name}" type="system">
       <hardware>
@@ -27,13 +30,19 @@
       </hardware>
       <!-- Pivot Joints -->
-      <joint name="${prefix}axle_yaw_front_joint">
-        <state_interface name="position" />
-      </joint>
+      <xacro:unless value="${lock_front_yaw}">
+        <joint name="${prefix}axle_yaw_front_joint">
+          <state_interface name="position" />
+        </joint>
+      </xacro:unless>
+      <xacro:unless value="${lock_back_yaw}">
       <joint name="${prefix}axle_yaw_back_joint">
           <state_interface name="position" />
-      </joint>
-      <joint name="${prefix}axle_roll_front_joint">
-          <state_interface name="position" />
-      </joint>
+        </joint>
+      </xacro:unless>
+      <xacro:unless value="${lock_front_roll}">
+        <joint name="${prefix}axle_roll_front_joint">
+            <state_interface name="position" />
+        </joint>
+      </xacro:unless>
       <!-- Wheel Joints -->
       <joint name="${prefix}wheel_front_left_joint">

File: zoe2_description/urdf/zoe2/zoe2_macro.xacro (robot description, xacro)
@@ -11,5 +11,10 @@
   <xacro:include filename="$(find zoe2_description)/urdf/zoe2/parts/antenna.xacro" />
   <xacro:include filename="$(find zoe2_description)/urdf/zoe2/zoe2_params.xacro" />
-  <xacro:macro name="zoe2" params="prefix *origin">
+  <xacro:macro name="zoe2" params="
+                prefix
+                lock_front_yaw:=false
+                lock_front_roll:=false
+                lock_back_yaw:=false
+                ">
     <!-- LINKS -->
     <link name = "${prefix}base_link">
@@ -59,18 +64,37 @@
         <origin xyz="0 ${antenna_location} ${chassis_height}" />
     </joint>
-    <joint name="${prefix}axle_roll_front_joint" type="revolute">
-        <parent link="${prefix}chassis" />
-        <child link="${prefix}front_roll" />
-        <origin xyz="0 ${(robot_length/2 - robot_hinge_length)} ${wheel_radius-base_link_height}" />
-        <limit lower="-0.5" upper="0.5" effort="10" velocity="10"/>
-        <axis xyz="0 1 0" />
-    </joint>
-    <joint name="${prefix}axle_yaw_front_joint" type="revolute">
-        <parent link="${prefix}front_roll" />
-        <child link="${prefix}front_axle" />
-        <origin xyz="0 ${robot_hinge_length} 0" />
-        <axis xyz="0 0 1"/>
-        <limit lower="${-front_vertical_limit}" upper="${front_vertical_limit}" effort="10" velocity="10"/>
-    </joint>
+    <xacro:unless value="${lock_front_roll}">
+        <joint name="${prefix}axle_roll_front_joint" type="revolute">
+            <parent link="${prefix}chassis" />
+            <child link="${prefix}front_roll" />
+            <origin xyz="0 ${(robot_length/2 - robot_hinge_length)} ${wheel_radius-base_link_height}" />
+                <limit lower="-0.5" upper="0.5" effort="10" velocity="10"/>
+                <axis xyz="0 1 0" />
+        </joint>
+    </xacro:unless>
+    <xacro:if value="${lock_front_roll}">
+        <joint name="${prefix}axle_roll_front_joint" type="fixed">
+            <parent link="${prefix}chassis" />
+            <child link="${prefix}front_roll" />
+            <origin xyz="0 ${(robot_length/2 - robot_hinge_length)} ${wheel_radius-base_link_height}" />
+        </joint>
+    </xacro:if>
+    <!--  if lock_front_yaw, make this fixed -->
+    <xacro:if value="${lock_front_yaw}">
+        <joint name="${prefix}axle_yaw_front_joint" type="fixed">
+            <parent link="${prefix}front_roll" />
+            <child link="${prefix}front_axle" />
+            <origin xyz="0 ${robot_hinge_length} 0" />
+        </joint>
+    </xacro:if>
+    <xacro:unless value="${lock_front_yaw}">
+        <joint name="${prefix}axle_yaw_front_joint" type="revolute">
+            <parent link="${prefix}front_roll" />
+            <child link="${prefix}front_axle" />
+            <origin xyz="0 ${robot_hinge_length} 0" />
+            <axis xyz="0 0 1"/>
+            <limit lower="${-front_vertical_limit}" upper="${front_vertical_limit}" effort="10" velocity="10"/>
+        </joint>
+    </xacro:unless>
     <joint name="${prefix}wheel_front_right_joint" type="continuous">
         <parent link="${prefix}front_axle" />
@@ -85,11 +109,20 @@
         <axis xyz="-1 0 0" />
     </joint>
-    <joint name="${prefix}axle_yaw_back_joint" type="revolute">
-        <parent link="${prefix}back_roll" />
-        <child link="${prefix}back_axle" />
-        <origin xyz="0 ${-robot_hinge_length} 0" />
-        <limit lower="${-front_vertical_limit}" upper="${front_vertical_limit}" effort="10" velocity="10"/>
-        <axis xyz="0 0 1"/>
-    </joint>
+    <xacro:unless value="${lock_back_yaw}">
+        <joint name="${prefix}axle_yaw_back_joint" type="revolute">
+            <parent link="${prefix}back_roll" />
+            <child link="${prefix}back_axle" />
+            <origin xyz="0 ${-robot_hinge_length} 0" />
+            <limit lower="${-front_vertical_limit}" upper="${front_vertical_limit}" effort="10" velocity="10"/>
+            <axis xyz="0 0 1"/>
+        </joint>
+    </xacro:unless>
+    <xacro:if value="${lock_back_yaw}">
+        <joint name="${prefix}axle_yaw_back_joint" type="fixed">
+            <parent link="${prefix}back_roll" />
+            <child link="${prefix}back_axle" />
+            <origin xyz="0 ${-robot_hinge_length} 0" />
+        </joint>
+    </xacro:if>
     <joint name="${prefix}wheel_back_right_joint" type="continuous">
         <parent link="${prefix}back_axle" />
